File: Hardware/PCB/flynn_mainboard/flynn_mainboard.kicad_sch (KiCad schematic)
At the start: 4 parts, among them J4 Conn_01x03, J5 Conn_02x20_Odd_Even, J6 Conn_01x03, J7 Conn_01x06

Commit message: version rooté
Parts:
- removed J4, J6: Conn_01x03, symbol Connector_Generic:Conn_01x03
- added C17: 330u, Capacitor_SMD:CP_Elec_6.3x5.4, symbol Device:C_Polarized
- added C18, C8: 100n, Capacitor_SMD:C_0603_1608Metric, symbol Device:C_Small
- added D4, D5: LED, LED_SMD:LED_0603_1608Metric, symbol Device:LED
- added H1, H3, H5, H7: MountingHole_Pad, MountingHole:MountingHole_2.7mm_M2.5_Pad, symbol Mechanical:MountingHole_Pad
- added J2: Conn_01x02, Connector_JST:JST_EH_B2B-EH-A_1x02_P2.50mm_Vertical, symbol Connector_Generic:Conn_01x02
- added R6, R8: 6.8k, Resistor_SMD:R_0603_1608Metric, symbol Device:R
- J5: value Conn_02x20_Odd_Even -> Rpi 2W Zéro; footprint (none) -> Connector_PinSocket_2.54mm:PinSocket_2x20_P2.54mm_Vertical
- J7: footprint (none) -> Connector_JST:JST_PH_B6B-PH-K_1x06_P2.00mm_Vertical
Connections:
- net +3.3V: now also J7.6 (Pin_6), C8.2, R8.1; no longer J7.1 (Pin_1)
- net DIR1: now also J5.22 (Pin_22), J5.32 (Pin_32); no longer J5.16 (Pin_16), J5.31 (Pin_31)
- net DIR2: now also J5.31 (Pin_31)
- net GND: now also J7.1 (Pin_1), C17.2, C18.2, C8.1, D4.1 (K), D5.1 (K), H1.1, H3.1, H5.1, H7.1, J2.1 (Pin_1); no longer J7.6 (Pin_6)
- net MISO: now also J5.21 (Pin_21); no longer J5.19 (Pin_19)
- net MOSI: now also J5.19 (Pin_19); no longer J5.40 (Pin_40)
- net STEP2: now also J5.33 (Pin_33)
- net STEP1: no longer names the net of J5.18 (Pin_18)
- net STEP1: no longer J5.29 (Pin_29)
- new net: D5.2 (A), R8.2
- new net: D4.2 (A), R6.2
- new net VCC: C17.1, C18.1, J2.2 (Pin_2), R6.1
Other:
- removed sheet TMC2225_COPIE
- added sheet tmc2225_driver1 (tmc2225_driverkicad_sch.kicad_sch)
- sheet tmc2225_driver ports: added DIR, STEP; removed none
- note added: "BATTERY"
- note added: "FIXING HOLES"
- note added: "LED"
- note added: "MCP3208 CONNECTOR"
- moved on the sheet: J5, J7
