File: Hardware/PCB/flynn_mainboard/lms6dsox.kicad_sch (KiCad schematic)
At the start: 0 parts

Commit message: Ajout du schéma
Parts:
- added C10, C11: 100nF, symbol Device:C_Small
- added R13: 10 K, symbol Device:R_Small
- added R14: 10K, symbol Device:R_Small
- added U4: LSM6DSOX, LSM6DSOX:PQFN50P250X300X86-14N, symbol LSM6DSOX:LSM6DSOX
Connections:
- new net +3.3V: C10.1, C11.2, R13.1, R14.1, U4.12 (CS), U4.5 (VDDIO), U4.8 (VDD)
- new net GND: C10.2, C11.1, U4.1 (SDO/SA0), U4.2 (SDX), U4.3 (SCX), U4.6 (GND), U4.7 (GND)
- new net SCL: R14.2, U4.13 (SCL)
- new net SDA: R13.2, U4.14 (SDA)
- no-connect marks 0 -> 4
Other:
- note added: "accelerometer"

Commit message: version rooté
Parts:
- added R19: 10k, Resistor_SMD:R_0603_1608Metric, symbol Device:R_Small
- C10, C11: footprint (none) -> Capacitor_SMD:C_0603_1608Metric
- R13, R14: footprint (none) -> Resistor_SMD:R_0603_1608Metric
- U4: footprint LSM6DSOX:PQFN50P250X300X86-14N -> Package_LGA:LGA-14_3x2.5mm_P0.5mm_LayoutBorder3x4y
Connections:
- net +3.3V: now also R19.1; no longer U4.12 (CS)
- new net: R19.2, U4.12 (CS)
Other:
- moved on the sheet: C10, C11, R13, R14, U4
