File: Hardware/PCB/flynn_mainboard/tmc2225_driverkicad_sch.kicad_sch (KiCad schematic)
At the start: 25 parts, among them J1 Conn_01x04, J2 Conn_01x02, SW1 SW_DIP_x02, U2 AZ1117-3.3

Commit message: version rooté
Parts:
- removed C2: 100n, symbol Device:C
- removed C4: 10u, symbol Device:C
- removed C6: 22u, symbol Device:C
- removed D2, D3: LED, symbol Device:LED
- removed H1, H3, H5, H7: MountingHole_Pad, symbol Mechanical:MountingHole_Pad
- removed J2: Conn_01x02, symbol Connector_Generic:Conn_01x02
- removed R2, R4: R, symbol Device:R
- removed SW1: SW_DIP_x02, symbol Switch:SW_DIP_x02
- removed U2: AZ1117-3.3, symbol Regulator_Linear:AZ1117-3.3
- added C15, C2, C6: 100n, Capacitor_SMD:C_0603_1608Metric, symbol Device:C_Small
- added R17, R2: R_Small, Resistor_SMD:R_0603_1608Metric, symbol Device:R_Small
- C1, C3, C5: footprint (none) -> Capacitor_SMD:C_0603_1608Metric
- D1: footprint (none) -> LED_SMD:LED_0603_1608Metric
- J1: footprint (none) -> Connector_JST:JST_PH_B4B-PH-K_1x04_P2.00mm_Vertical
- R1, R3: value 150m -> 220m; footprint (none) -> Resistor_SMD:R_1206_3216Metric
- R5, R7, R9: footprint (none) -> Resistor_SMD:R_0603_1608Metric
- U1: footprint (none) -> Package_SO:HTSSOP-28-1EP_4.4x9.7mm_P0.65mm_EP2.85x5.4mm_ThermalVias
Connections:
- net VCC is gone; now on net GND: C3.1, U1.11 (VS), U1.4 (VS)
- net +3.3V: now also C15.1, R17.1, R2.1
- net GND: now also C15.2, C2.1, C2.2, C6.1, C6.2
- net at R9.1, U1.25 (MS1): now also R2.2
- net at R7.1, U1.26 (MS2): now also R17.2
- net DIR1 renamed DIR
- net STEP1 renamed STEP
Other:
- note removed: "Supply"
- moved on the sheet: C1, C3, C5, D1, J1, R1, R3, R5, R7, R9, U1
