File: Hardware/PCB/flynn_mainboard/tmc2225_driverkicad_sch.kicad_sch (KiCad schematic)
At the start: 0 parts

Commit message: Update README & JOURNALING
Parts:
- added C1: 22n, symbol Device:C_Small
- added C2: 100n, symbol Device:C
- added C3: 100n, symbol Device:C_Small
- added C4: 10u, symbol Device:C
- added C5: 2u2, symbol Device:C_Small
- added C6: 22u, symbol Device:C
- added D1, D2, D3: LED, symbol Device:LED
- added H1, H3, H5, H7: MountingHole_Pad, symbol Mechanical:MountingHole_Pad
- added J1: Conn_01x04, symbol Connector_Generic:Conn_01x04
- added J2: Conn_01x02, symbol Connector_Generic:Conn_01x02
- added R1, R3: 150m, symbol Device:R_Small
- added R2, R4: R, symbol Device:R
- added R5: 1k, symbol Device:R_Small
- added R7, R9: 10K, symbol Device:R_Small
- added SW1: SW_DIP_x02, symbol Switch:SW_DIP_x02
- added U1: ~, symbol my_lib:TMC2225
- added U2: AZ1117-3.3, symbol Regulator_Linear:AZ1117-3.3
Connections:
- new net: J1.1 (Pin_1), U1.5 (OA2)
- new net: J1.2 (Pin_2), U1.7 (OA1)
- new net: J1.3 (Pin_3), U1.8 (OB1)
- new net: J1.4 (Pin_4), U1.10 (OB2)
- new net: C5.1, U1.15 (5VOUT)
- new net: D3.2 (A), R4.2
- new net: D2.2 (A), R2.2
- new net: C1.1, U1.1 (CPO)
- new net: R5.1, U1.18 (DIAG)
- new net: C1.2, U1.2 (CPI)
- new net: R9.1, SW1.3, U1.25 (MS1)
- new net: R7.1, SW1.4, U1.26 (MS2)
- new net: C3.2, U1.3 (VCP)
- new net: R1.1, U1.6 (BRA)
- new net: R3.1, U1.9 (BRB)
- new net: D1.2 (A), R5.2
- new net +3.3V: C6.1, R4.1, SW1.1, SW1.2, U1.16 (VCC_IO), U2.2 (VO)
- new net DIR1: U1.20 (DIR)
- new net GND: C2.2, C4.2, C5.2, C6.2, D1.1 (K), D2.1 (K), D3.1 (K), H1.1, H3.1, H5.1, H7.1, J2.1 (Pin_1), R1.2, R3.2, R7.2, R9.2, U1.13 (TEST), U1.14 (GND), U1.21 (ENN), U1.28 (GND), U1.29 (PAD), U2.1 (GND)
- new net STEP1: U1.22 (STEP)
- new net VCC: C2.1, C3.1, C4.1, J2.2 (Pin_2), R2.1, U1.11 (VS), U1.4 (VS), U2.3 (VI)
- no-connect marks 0 -> 1
Other:
- note added: "Driver + motor connectors"
- note added: "Supply"
- title: (none) -> Flynn

Commit message: Journaling Update
Parts:
- removed C2: 100n, symbol Device:C
- removed C4: 10u, symbol Device:C
- removed C6: 22u, symbol Device:C
- removed D2, D3: LED, symbol Device:LED
- removed H1, H3, H5, H7: MountingHole_Pad, symbol Mechanical:MountingHole_Pad
- removed J2: Conn_01x02, symbol Connector_Generic:Conn_01x02
- removed R2, R4: R, symbol Device:R
- removed SW1: SW_DIP_x02, symbol Switch:SW_DIP_x02
- removed U2: AZ1117-3.3, symbol Regulator_Linear:AZ1117-3.3
- added C15, C2, C6: 100n, Capacitor_SMD:C_0603_1608Metric, symbol Device:C_Small
- added R17, R2: R_Small, Resistor_SMD:R_0603_1608Metric, symbol Device:R_Small
- C1, C3, C5: footprint (none) -> Capacitor_SMD:C_0603_1608Metric
- D1: footprint (none) -> LED_SMD:LED_0603_1608Metric
- J1: footprint (none) -> Connector_JST:JST_PH_B4B-PH-K_1x04_P2.00mm_Vertical
- R1, R3: value 150m -> 220m; footprint (none) -> Resistor_SMD:R_1206_3216Metric
- R5, R7, R9: footprint (none) -> Resistor_SMD:R_0603_1608Metric
- U1: footprint (none) -> Package_SO:HTSSOP-28-1EP_4.4x9.7mm_P0.65mm_EP2.85x5.4mm_ThermalVias
Connections:
- net VCC is gone; now on net GND: C3.1, U1.11 (VS), U1.4 (VS)
- net +3.3V: now also C15.1, R17.1, R2.1
- net GND: now also C15.2, C2.1, C2.2, C6.1, C6.2
- net at R9.1, U1.25 (MS1): now also R2.2
- net at R7.1, U1.26 (MS2): now also R17.2
- net DIR1 renamed DIR
- net STEP1 renamed STEP
Other:
- note removed: "Supply"
- moved on the sheet: C1, C3, C5, D1, J1, R1, R3, R5, R7, R9, U1
