File: flynn_mainboard/flynn_mainboard.kicad_pcb (KiCad board)
At the start: 4 copper layers, 65 x 30 mm, 52 parts, among them J1 Conn_01x04, J2 Conn_01x02, J4 Conn_01x04, J5 Rpi 2W Zéro, J7 Conn_01x06, U4 LSM6DSOX

Commit message: Add files via upload
Parts:
- removed J5: Rpi 2W Zéro, Connector_PinSocket_2.54mm:PinSocket_2x20_P2.54mm_Vertical
- added J103: Rpi 2W Zéro, Connector_PinSocket_2.54mm:PinSocket_2x20_P2.54mm_Vertical, B.Cu at (104.9, 101.0)
- moved C404 10.2 mm to (106.0, 115.9)
- moved C205 10.1 mm to (153.1, 116.1), turned to 0 degrees
- moved C401 6.49 mm to (106.9, 105.7), turned to 0 degrees
- moved R401 4.16 mm to (118.5, 110.3), turned to 180 degrees
- moved R203 4.03 mm to (140.5, 116.9), turned to 0 degrees
- moved R202 3.35 mm to (140.5, 113.8), turned to 180 degrees
- moved R404 2.94 mm to (118.5, 105.8)
- moved C204 1.74 mm to (152.0, 107.7), turned to 0 degrees
- moved R204 1.68 mm to (140.5, 115.4), turned to 180 degrees
- moved R402 1.46 mm to (118.5, 108.8)
- moved R403 1.28 mm to (118.5, 107.3), turned to 180 degrees
- moved R301 1.20 mm to (124.6, 109.2), turned to 0 degrees
- moved C201 1.13 mm to (153.5, 118.8)
- moved C202 1.13 mm to (152.0, 118.8)
- moved R201 0.86 mm to (140.5, 112.3), turned to 0 degrees
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- renumbered C8 to C101, C17 to C102, C18 to C103, C3 to C201, C1 to C202, C15 to C203, C2 to C204, C6 to C205, C5 to C206, C10 to C301, C11 to C302, C12 to C401, C13 to C402, C16 to C403, C4 to C404, C7 to C405, C14 to C406, D4 to D101, D5 to D102, D1 to D201, D6 to D401, H3 to H101, H1 to H102, H5 to H103, H7 to H104, J2 to J101, J7 to J102, J1 to J201, J4 to J401, R6 to R101, R8 to R102, R2 to R201, R9 to R202, R17 to R203, R7 to R204, R1 to R205, R3 to R206, R5 to R207, R13 to R301, R14 to R302, R19 to R303, R4 to R401, R10 to R402, R18 to R403, R11 to R404, R12 to R405, R15 to R406, R16 to R407, U1 to U201, U4 to U301, U5 to U401
Routing:
- net VCC: track 44.9 -> 26.6 mm, vias 5 -> 9
- net GND: track 8.00 -> 25.3 mm, vias 6 -> 30
- net Net-(U201-MS2): track 12.6 -> 3.47 mm, vias 2 -> 0
- net +3.3V: track 47.6 -> 40.4 mm, vias 10 -> 12
- net Net-(U401-MS1): track 7.50 -> 3.17 mm
- net Net-(U201-MS1): track 7.24 -> 3.94 mm
- net SDA: track 27.0 -> 25.6 mm
- net Net-(U401-MS2): track 4.42 -> 3.46 mm
- net Net-(D201-A): track 1.52 -> 2.23 mm
- net Net-(U201-VCP): track 5.92 -> 6.50 mm
- net Net-(U401-VCP): track 4.66 -> 4.13 mm
- net Net-(U201-CPI): track 4.15 -> 4.66 mm
