File: flynn_mainboard/flynn_mainboard.kicad_sch (KiCad schematic)
At the start: 14 parts, among them J2 Conn_01x02, J5 Rpi 2W Zéro, J7 Conn_01x06

Commit message: Add files via upload
Parts:
- renumbered C8 to C101, C17 to C102, C18 to C103, D4 to D101, D5 to D102, H3 to H101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
Connections:
- net +5V: no longer names the net of J103.2 (Pin_2)
- net +5V: no longer J103.4 (Pin_4)
- no-connect marks 18 -> 20
