File: flynn_mainboard/lms6dsox.kicad_sch (KiCad schematic)
At the start: 6 parts, among them U4 LSM6DSOX

Commit message: Add files via upload
Parts:
- renumbered C10 to C301, C11 to C302, R13 to R301, R14 to R302, R19 to R303, U4 to U301
Changed lines of the file:
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@@
 		(dnp no)
 		(fields_autoplaced yes)
-		(property "Reference" "#PWR037"
+		(property "Reference" "#PWR0304"
 			(at 173.99 88.9 0)
 			(effects
@@
 			(project "flynn_mainboard"
 				(path "/56ec65ab-c401-455a-8a7c-6731af93b01f/62427f22-d6cc-475c-bb62-0af0fcc02fef"
-					(reference "#PWR037")
+					(reference "#PWR0304")
 					(unit 1)
 				)
@@
 		(dnp no)
 		(fields_autoplaced yes)
-		(property "Reference" "#PWR035"
+		(property "Reference" "#PWR0302"
 			(at 119.38 71.12 0)
 			(effects
@@
 			(project "flynn_mainboard"
 				(path "/56ec65ab-c401-455a-8a7c-6731af93b01f/62427f22-d6cc-475c-bb62-0af0fcc02fef"
-					(reference "#PWR035")
+					(reference "#PWR0302")
 					(unit 1)
 				)
@@
 		(dnp no)
 		(fields_autoplaced yes)
-		(property "Reference" "#PWR038"
+		(property "Reference" "#PWR0305"
 			(at 173.99 109.22 0)
 			(effects
@@
 			(project "flynn_mainboard"
 				(path "/56ec65ab-c401-455a-8a7c-6731af93b01f/62427f22-d6cc-475c-bb62-0af0fcc02fef"
-					(reference "#PWR038")
+					(reference "#PWR0305")
 					(unit 1)
 				)
@@
 		(dnp no)
 		(fields_autoplaced yes)
-		(property "Reference" "#PWR034"
+		(property "Reference" "#PWR0301"
 			(at 109.22 72.39 0)
 			(effects
@@
 			(project "flynn_mainboard"
 				(path "/56ec65ab-c401-455a-8a7c-6731af93b01f/62427f22-d6cc-475c-bb62-0af0fcc02fef"
-					(reference "#PWR034")
+					(reference "#PWR0301")
 					(unit 1)
 				)
@@
 		(dnp no)
 		(fields_autoplaced yes)
-		(property "Reference" "R14"
+		(property "Reference" "R302"
 			(at 121.92 71.1199 0)
 			(effects
@@
 			(project "flynn_mainboard"
 				(path "/56ec65ab-c401-455a-8a7c-6731af93b01f/62427f22-d6cc-475c-bb62-0af0fcc02fef"
-					(reference "R14")
+					(reference "R302")
 					(unit 1)
 				)
@@
 		(on_board yes)
 		(dnp no)
-		(property "Reference" "#PWR042"
+		(property "Reference" "#PWR0308"
 			(at 195.58 81.28 0)
 			(effects
@@
 			(project "flynn_mainboard"
 				(path "/56ec65ab-c401-455a-8a7c-6731af93b01f/62427f22-d6cc-475c-bb62-0af0fcc02fef"
-					(reference "#PWR042")
+					(reference "#PWR0308")
 					(unit 1)
 				)
@@
 		(dnp no)
 		(fields_autoplaced yes)
-		(property "Reference" "#PWR041"
+		(property "Reference" "#PWR0307"
 			(at 193.04 88.9 0)
 			(effects
@@
 			(project "flynn_mainboard"
 				(path "/56ec65ab-c401-455a-8a7c-6731af93b01f/62427f22-d6cc-475c-bb62-0af0fcc02fef"
-					(reference "#PWR041")
+					(reference "#PWR0307")
 					(unit 1)
 				)
@@
 		(on_board yes)
 		(dnp no)
-		(property "Reference" "R19"
+		(property "Reference" "R303"
 			(at 129.54 74.9299 0)
 			(effects
@@
 			(project ""
 				(path "/56ec65ab-c401-455a-8a7c-6731af93b01f/62427f22-d6cc-475c-bb62-0af0fcc02fef"
-					(reference "R19")
+					(reference "R303")
 					(unit 1)
 				)
@@
 		(on_board yes)
 		(dnp no)
-		(property "Reference" "#PWR036"
+		(property "Reference" "#PWR0303"
 			(at 132.08 72.39 0)
 			(effects
@@
 			(project "flynn_mainboard"
 				(path "/56ec65ab-c401-455a-8a7c-6731af93b01f/62427f22-d6cc-475c-bb62-0af0fcc02fef"
-					(reference "#PWR036")
+					(reference "#PWR0303")
 					(unit 1)
 				)
@@
 		(on_board yes)
 		(dnp no)
-		(property "Reference" "R13"
+		(property "Reference" "R301"
 			(at 105.41 74.422 0)
 			(effects
@@
 			(project "flynn_mainboard"
 				(path "/56ec65ab-c401-455a-8a7c-6731af93b01f/62427f22-d6cc-475c-bb62-0af0fcc02fef"
-					(reference "R13")
+					(reference "R301")
 					(unit 1)
 				)
@@
 		(dnp no)
 		(fields_autoplaced yes)
-		(property "Reference" "C10"
+		(property "Reference" "C301"
 			(at 182.88 81.9213 0)
 			(effects
@@
 			(project "flynn_mainboard"
 				(path "/56ec65ab-c401-455a-8a7c-6731af93b01f/62427f22-d6cc-475c-bb62-0af0fcc02fef"
-					(reference "C10")
+					(reference "C301")
 					(unit 1)
 				)
@@
 		(dnp no)
 		(fields_autoplaced yes)
-		(property "Reference" "#PWR040"
+		(property "Reference" "#PWR0306"
 			(at 180.34 91.44 0)
 			(effects
@@
 			(project "flynn_mainboard"
 				(path "/56ec65ab-c401-455a-8a7c-6731af93b01f/62427f22-d6cc-475c-bb62-0af0fcc02fef"
-					(reference "#PWR040")
+					(reference "#PWR0306")
 					(unit 1)
 				)
@@
 		(dnp no)
 		(fields_autoplaced yes)
-		(property "Reference" "U4"
+		(property "Reference" "U301"
 			(at 149.86 71.12 0)
 			(effects
@@
 			(project "flynn_mainboard"
 				(path "/56ec65ab-c401-455a-8a7c-6731af93b01f/62427f22-d6cc-475c-bb62-0af0fcc02fef"
-					(reference "U4")
+					(reference "U301")
 					(unit 1)
 				)
@@
 		(dnp no)
 		(fields_autoplaced yes)
-		(property "Reference" "C11"
+		(property "Reference" "C302"
 			(at 195.58 79.3686 0)
 			(effects
@@
 			(project "flynn_mainboard"
 				(path "/56ec65ab-c401-455a-8a7c-6731af93b01f/62427f22-d6cc-475c-bb62-0af0fcc02fef"
-					(reference "C11")
-					(unit 1)
-				)
+					(reference "C302")
+					(unit 1)
+				)
