File: flynn_mainboard/tmc2225_driverkicad_sch.kicad_sch (KiCad schematic)
At the start: 16 parts, among them J1 Conn_01x04

Commit message: Add files via upload
Parts:
- renumbered C3 to C201, C1 to C202, C15 to C203, C2 to C204, C6 to C205, C5 to C206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
