File: 2526_B3_S6_Projet_Flynn/Hardware/PCB/flynn_mainboard/flynn_mainboard.kicad_sch (KiCad schematic)
At the start: 14 parts, among them J101 Conn_01x02, J102 Conn_01x06, J103 Rpi 2W Zéro

Commit message: Add files via upload
Other:
- note added: "2 RED LED"
Changed lines of the file:
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@@
+		)
+	)
+	(text "2 RED LED\n"
+		(exclude_from_sim no)
+		(at 96.012 154.686 0)
+		(effects
+			(font
+				(size 1.27 1.27)
+			)
 		)
 	)
@@
 		)
 	)
-	(text "MCP3208 CONNECTOR"
+	(text "LED"
 		(exclude_from_sim no)
-		(at 26.416 94.742 0)
+		(at 75.946 141.732 0)
 		(effects
 			(font
@@
 		)
 	)
-	(text "LED\n"
+	(text "MCP3208 CONNECTOR"
 		(exclude_from_sim no)
-		(at 76.454 142.24 0)
+		(at 26.416 94.742 0)
 		(effects
 			(font
